File: pcb/console/console.kicad_pcb (KiCad board)
At the start: 2 copper layers, 80 x 60 mm, 6 parts, among them J1 Micro_SD_Card, U1 RP2040-ZERO

Commit message: Final PCB design
Parts:
- J1: value Micro_SD_Card -> SD Card; footprint Connector_Card:microSD_HC_Wuerth_693072010801 -> footprints:TF-015
- moved J1 9.40 mm to (227.7, 37.0), turned to -90 degrees
- renumbered A1 to A, B1 to B, Brd1 to Screen
Routing:
- net GND: track 197.9 -> 0.00 mm, vias 3 -> 0
- net /CS: track 77.3 -> 62.4 mm
- net /SCLK: track 73.3 -> 60.5 mm
- net +3.3V: track 56.9 -> 45.2 mm
- net /MOSI: track 71.5 -> 60.6 mm
- net /MISO: track 75.5 -> 65.3 mm
- net /B: track 65.9 -> 72.1 mm
- net /SCL0: track 40.2 -> 43.9 mm
- net /RIGHT: track 35.5 -> 38.6 mm
- net /DOWN: track 45.4 -> 42.7 mm
- net /LEFT: track 25.0 -> 25.9 mm
- net /SDA0: track 47.2 -> 46.5 mm
- net /A: track 63.2 -> 63.8 mm
