File: pcb/console/console.kicad_sch (KiCad schematic)
At the start: 6 parts, among them J1 Micro_SD_Card, U1 RP2040-ZERO

Commit message: Final PCB design
Parts:
- J1: footprint Connector_Card:microSD_HC_Wuerth_693072010801 -> footprints:TF-015
Changed lines of the file:
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@@
 			)
 		)
-		(property "Footprint" "Connector_Card:microSD_HC_Wuerth_693072010801"
+		(property "Footprint" "footprints:TF-015"
 			(at 175.26 124.46 0)
 			(effects
